File: eagle/lpc134x.brd (EAGLE design)
At the start: 39.8 x 24.7 mm, 35 parts, among them IC2 LT1763CS8-3.3, Q1 12Mhz, SW1 SWITCH_MCTAEF, T1 Si2301DS, X1 USB-MICROB

Commit message: updates
Parts:
- added U$1: (no value), seb:C3D2_LOGO
- added U$2: (no value), seb:C3D2_LOGO_SMALL
- C2: value 100nF -> 22pF
- C3: value 22pF -> 100nF
- R1: value 15k -> 1k5
- R9: value 1k5 -> 15k
- moved R10 11.2 mm to (11.1, 14.5), turned to 180 degrees
- moved R9 6.02 mm to (5.12, 5.00)
- moved R1 5.20 mm to (10.4, 9.32), turned to 0 degrees
- moved C2 3.80 mm to (14.9, 6.28), turned to 0 degrees
- moved C3 3.80 mm to (18.4, 7.97), turned to 90 degrees
- moved R8 3.09 mm to (8.12, 5.62), turned to 270 degrees
- moved T1 2.00 mm to (11.1, 6.38)
- moved R5 1.38 mm to (10.4, 10.9)
- moved R4 1.01 mm to (10.4, 12.3)
- moved C10 0.12 mm to (6.00, 12.0)
- moved C9 0.12 mm to (6.00, 8.88)
Connections:
- net +3V3: now also C3.2, R10.2; no longer C2.2, R1.2
- net +5V: now also R9.1; no longer R10.1
- net N$10: now also R1.1; no longer R9.1
- net N$20: now also R1.2; no longer R9.2
- net N$3: now also C2.2; no longer C3.2
- net RST: now also R10.1; no longer R1.1
- net VBUS: now also R9.2; no longer R10.2
Routing:
- net +3V3: track 76.7 -> 75.2 mm
- net 01: track 15.0 -> 13.8 mm
- net 06: track 21.0 -> 20.1 mm
- net N$20: track 2.67 -> 1.85 mm
- net N$10: track 7.74 -> 8.33 mm
- net N$11: track 6.38 -> 6.96 mm
- net GND: vias 35 -> 30
