File: eagle/lpc134x.sch (EAGLE design)
At the start: 35 parts, among them IC2 LT1763CS8-3.3, Q1 12Mhz, SW1 SWITCH_MCTAEF, T1 Si2301DS, X1 USB-MICROB

Commit message: updates
Parts:
- C2: value 100nF -> 22pF
- C3: value 22pF -> 100nF
- R1: value 15k -> 1k5
- R9: value 1k5 -> 15k
Connections:
- net +3V3: now also C3.2, R10.2; no longer C2.2, R1.2
- net +5V: now also R9.1; no longer R10.1
- net N$10: now also R1.1; no longer R9.1
- net N$20: now also R1.2; no longer R9.2
- net N$3: now also C2.2; no longer C3.2
- net RST: now also R10.1; no longer R1.1
- net VBUS: now also R9.2; no longer R10.2
Other:
- moved on the sheet: C2, C3, R1, R10, R9
Changed lines of the file:
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@@
 <part name="+3V2" library="supply1" deviceset="+3V3" device=""/>
 <part name="+3V4" library="supply1" deviceset="+3V3" device=""/>
-<part name="R1" library="rcl" deviceset="R-EU_" device="R0402" value="15k"/>
+<part name="R10" library="rcl" deviceset="R-EU_" device="R0402" value="15k"/>
 <part name="JP1" library="pinhead-2" deviceset="PINHD-1X10" device="_2.54"/>
 <part name="JP2" library="pinhead-2" deviceset="PINHD-1X10" device="_2.54"/>
@@
 <part name="BL/SW2" library="seb" deviceset="SWITCH_MCTAEF" device=""/>
 <part name="SW1" library="seb" deviceset="SWITCH_MCTAEF" device=""/>
-<part name="C3" library="rcl" deviceset="C-EU" device="C0402" value="22pF"/>
+<part name="C2" library="rcl" deviceset="C-EU" device="C0402" value="22pF"/>
 <part name="C1" library="rcl" deviceset="C-EU" device="C0402" value="22pF"/>
-<part name="C2" library="rcl" deviceset="C-EU" device="C0402" value="100nF"/>
+<part name="C3" library="rcl" deviceset="C-EU" device="C0402" value="100nF"/>
 <part name="C4" library="rcl" deviceset="C-EU" device="C0402" value="100nF"/>
 <part name="R6" library="rcl" deviceset="R-EU_" device="R0402" value="150R"/>
 <part name="R7" library="rcl" deviceset="R-EU_" device="R0402" value="150R"/>
 <part name="Q1" library="seb" deviceset="MT-OSCILLATOR" device="" value="12Mhz"/>
-<part name="R9" library="rcl" deviceset="R-EU_" device="R0402" value="1k5"/>
+<part name="R1" library="rcl" deviceset="R-EU_" device="R0402" value="1k5"/>
 <part name="IC2" library="linear-technology" deviceset="LT1763CS8" device="" technology="-3.3"/>
 <part name="C5" library="SparkFun" deviceset="CAP" device="0805" value="1µF"/>
@@
 <part name="P+5" library="supply1" deviceset="+5V" device=""/>
 <part name="R8" library="rcl" deviceset="R-EU_" device="R0402" value="15k"/>
-<part name="R10" library="rcl" deviceset="R-EU_" device="R0402" value="15k"/>
+<part name="R9" library="rcl" deviceset="R-EU_" device="R0402" value="15k"/>
 <part name="P+1" library="supply1" deviceset="+5V" device=""/>
 <part name="GND11" library="supply1" deviceset="GND" device=""/>
@@
 <instance part="+3V2" gate="G$1" x="-73.66" y="271.78"/>
 <instance part="+3V4" gate="G$1" x="177.8" y="144.78" rot="R180"/>
-<instance part="R1" gate="G$1" x="177.8" y="154.94" rot="R270"/>
+<instance part="R10" gate="G$1" x="177.8" y="154.94" rot="R270"/>
 <instance part="JP1" gate="A" x="165.1" y="251.46" rot="R180"/>
 <instance part="JP2" gate="A" x="215.9" y="254" rot="MR0"/>
@@
 <attribute name="NAME" x="159.385" y="168.91" size="1.778" layer="95" rot="MR0"/>
 </instance>
-<instance part="C3" gate="G$1" x="-78.74" y="226.06" rot="R90"/>
+<instance part="C2" gate="G$1" x="-78.74" y="226.06" rot="R90"/>
 <instance part="C1" gate="G$1" x="-78.74" y="231.14" rot="R90"/>
-<instance part="C2" gate="G$1" x="-73.66" y="261.62" rot="R180"/>
+<instance part="C3" gate="G$1" x="-73.66" y="261.62" rot="R180"/>
 <instance part="C4" gate="G$1" x="-66.04" y="261.62" rot="R180"/>
 <instance part="R6" gate="G$1" x="251.46" y="254" rot="R180"/>
 <instance part="R7" gate="G$1" x="251.46" y="256.54" rot="R180"/>
 <instance part="Q1" gate="G$1" x="-68.58" y="228.6" rot="R90"/>
-<instance part="R9" gate="G$1" x="-73.66" y="180.34" rot="R270"/>
+<instance part="R1" gate="G$1" x="-73.66" y="180.34" rot="R270"/>
 <instance part="IC2" gate="G$1" x="193.04" y="210.82"/>
 <instance part="C5" gate="G$1" x="167.64" y="203.2"/>
@@
 </instance>
 <instance part="R8" gate="G$1" x="-43.18" y="254" rot="R90"/>
-<instance part="R10" gate="G$1" x="-43.18" y="264.16" rot="R270"/>
+<instance part="R9" gate="G$1" x="-43.18" y="264.16" rot="R270"/>
 <instance part="P+1" gate="1" x="-43.18" y="271.78"/>
 <instance part="GND11" gate="1" x="-43.18" y="246.38"/>
@@
 <wire x1="-73.66" y1="226.06" x2="-68.58" y2="226.06" width="0.1524" layer="91"/>
 <junction x="-68.58" y="226.06"/>
-<pinref part="C3" gate="G$1" pin="2"/>
+<pinref part="C2" gate="G$1" pin="2"/>
 <pinref part="Q1" gate="G$1" pin="1"/>
 <label x="-63.5" y="226.06" size="1.778" layer="95"/>
@@
 <junction x="-81.28" y="226.06"/>
 <pinref part="GND2" gate="1" pin="GND"/>
-<pinref part="C3" gate="G$1" pin="1"/>
+<pinref part="C2" gate="G$1" pin="1"/>
 <pinref part="C1" gate="G$1" pin="1"/>
 </segment>
@@
 <junction x="-73.66" y="256.54"/>
 <pinref part="GND3" gate="1" pin="GND"/>
-<pinref part="C2" gate="G$1" pin="1"/>
+<pinref part="C3" gate="G$1" pin="1"/>
 <pinref part="C4" gate="G$1" pin="1"/>
 </segment>
@@
 <wire x1="177.8" y1="149.86" x2="177.8" y2="147.32" width="0.1524" layer="91"/>
 <pinref part="+3V4" gate="G$1" pin="+3V3"/>
-<pinref part="R1" gate="G$1" pin="2"/>
+<pinref part="R10" gate="G$1" pin="2"/>
 </segment>
 <segment>
@@
 <wire x1="-73.66" y1="269.24" x2="-73.66" y2="266.7" width="0.1524" layer="91"/>
 <pinref part="+3V2" gate="G$1" pin="+3V3"/>
-<pinref part="C2" gate="G$1" pin="2"/>
+<pinref part="C3" gate="G$1" pin="2"/>
 <pinref part="C4" gate="G$1" pin="2"/>
 <wire x1="-73.66" y1="269.24" x2="-66.04" y2="269.24" width="0.1524" layer="91"/>
@@
 <wire x1="177.8" y1="162.56" x2="172.72" y2="162.56" width="0.1524" layer="91"/>
 <junction x="177.8" y="162.56"/>
-<pinref part="R1" gate="G$1" pin="1"/>
+<pinref part="R10" gate="G$1" pin="1"/>
 <pinref part="RST" gate="G$1" pin="2"/>
 <label x="180.34" y="162.56" size="1.778" layer="95"/>
@@
 </segment>
 <segment>
-<pinref part="R10" gate="G$1" pin="1"/>
+<pinref part="R9" gate="G$1" pin="1"/>
 <pinref part="P+1" gate="1" pin="+5V"/>
 </segment>
@@
 <junction x="-73.66" y="185.42"/>
 <pinref part="R5" gate="G$1" pin="2"/>
-<pinref part="R9" gate="G$1" pin="1"/>
+<pinref part="R1" gate="G$1" pin="1"/>
 <pinref part="C9" gate="G$1" pin="1"/>
 <wire x1="-83.82" y1="185.42" x2="-73.66" y2="185.42" width="0.1524" layer="91"/>
@@
 <segment>
 <wire x1="-73.66" y1="175.26" x2="-73.66" y2="172.72" width="0.1524" layer="91"/>
-<pinref part="R9" gate="G$1" pin="2"/>
+<pinref part="R1" gate="G$1" pin="2"/>
 <pinref part="T1" gate="G$1" pin="D"/>
 </segment>
@@
 <junction x="-43.18" y="259.08"/>
 <pinref part="R8" gate="G$1" pin="2"/>
-<pinref part="R10" gate="G$1" pin="2"/>
+<pinref part="R9" gate="G$1" pin="2"/>
 <label x="-38.1" y="259.08" size="1.778" layer="95"/>
 </segment>

Commit message: pcb update
Parts:
- removed C10, C9: 22pF, rcl:C-EUC0402
- removed JP5: (no value), pinhead:PINHD-1X1
- removed X1: USB-MICROB, SparkFun-Connectors:USB-MICROB
- added JP3: (no value), SparkFun-Connectors:M02PTH
- added X2: USB-SMD-NS, SparkFun-Connectors:USB-SMD-NS
- JP1: value (none) -> M10"; device pinhead-2:PINHD-1X10_2.54 -> SparkFun-Connectors:M10"
- JP2: device pinhead-2:PINHD-1X10_2.54 -> SparkFun-Connectors:M02PTH
- JP4: device pinhead-2:PINHD-1X02_2.54 -> SparkFun-Connectors:M02PTH
- JP6: value (none) -> M10"; device pinhead:PINHD-1X1 -> SparkFun-Connectors:M10"
- R1: value 1k5 -> 15k
- R10: value 15k -> 1k5
Connections:
- net N$14 renamed USB_D-
- net N$24 renamed USB_D+
- net N$3 renamed XTAL_OUT
- net N$4 renamed XTAL_IN
- net +3V3: now also JP3.1, JP3.2, R1.2; no longer JP5.1, R10.2
- net +5V: now also JP4.1, JP4.2, X2.VBUS; no longer JP6.1, X1.VBUS
- net 010: now also JP6.2; no longer JP1.2
- net 015: now also JP1.3; no longer JP2.8
- net 016: now also JP1.4; no longer JP2.7
- net 017: now also JP1.5; no longer JP2.6
- net 022: now also JP6.1; no longer JP1.1
- net 07: now also JP6.5; no longer JP1.5
- net 08: now also JP6.4; no longer JP1.4
- net 09: now also JP6.3; no longer JP1.3
- net 116: now also JP1.8; no longer JP2.3
- net 120: now also JP6.9; no longer JP1.9
- net 122: now also JP1.2; no longer JP2.9
- net 123: now also JP6.6; no longer JP1.6
- net 125: now also JP1.9; no longer JP2.2
- net 127: now also JP6.10; no longer JP1.10
- net GND: now also JP1.1, JP2.1, JP2.2, X2.GND; no longer C10.1, C9.2, JP2.10, JP4.1, JP4.2, X1.GND
- net N$10: now also R10.1, X2.D+; no longer C9.1, R1.1, X1.D+
- net N$11: now also X2.D-; no longer C10.2, X1.D-
- net N$20: now also R10.2; no longer R1.2
- net RST: now also JP1.10, R1.1; no longer JP2.1, R10.1
- net RX: now also JP1.6; no longer JP2.5
- net SCL: now also JP6.8; no longer JP1.8
- net SDA: now also JP6.7; no longer JP1.7
- net TX: now also JP1.7; no longer JP2.4
Other:
- note added: "<<</>>"
- note added: "Buttons"
- note added: "CC-BY-SA 3.0"
- note added: "Crystal"
- note added: "Dev-board"
- note added: "LEDs"
- note added: "LPC1347"
- note added: "Microcontroller"
- note added: "Pin Headers"
- note added: "Regulator"
- note added: "UART safety resitors"
- note added: "USB"
- note added: "VCC Capacitors"
- note added: "Voltage Divider for USB Detection"
- note added: "https://github.com/sebseb7/pentarm13uxx"
- note added: "seb@exse.net"
- moved on the sheet: BL/SW2, C1, C2, C3, C4, C5, C6, C7, C8, IC1, IC2, LED1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
